Commit message: March 19

File: urdf/scara.2nd.urdf (robot description, URDF)
Before this commit: robot scara, 5 links, 4 joints
Links:
- link base_link: mass None -> 5; geometry collision box size=0.223 0.12 0.238; visual mesh filename=package://scara_robot/meshes/base.STL scale=0.001 0.001 0.001
- link link1: mass None -> 2; geometry collision box size=0.35 0.1 0.05; visual mesh filename=package://scara_robot/meshes/link1.STL scale=0.001 0.001 0.001
- link link2: mass None -> 3; geometry collision box size=0.25 0.15 0.3; visual mesh filename=package://scara_robot/meshes/link2.STL scale=0.001 0.001 0.001
- link link3: mass None -> 0.1; geometry collision box size=0.04 0.025 0.219; visual mesh filename=package://scara_robot/meshes/link3.STL scale=0.001 0.001 0.001
- link link4: mass None -> 0.2; geometry collision box size=0.06 0.04 0.136456; visual mesh filename=package://scara_robot/meshes/link4.STL scale=0.001 0.001 0.001
Joints:
- joint base_to_link1: limit lower=-2.094395 upper=2.094395 effort=1000.0 velocity=0.2 -> lower=-2.094395 upper=2.094395 effort=1000.0 velocity=0.02
- joint link1_to_link2: limit lower=-2.268928 upper=2.268928 effort=1000.0 velocity=0.2 -> lower=-2.268928 upper=2.268928 effort=1000.0 velocity=0.02
- joint link2_to_link3: limit lower=-0.15 upper=0.0 effort=1000.0 velocity=0.002 -> lower=-0.15 upper=0.0 effort=1000.0 velocity=0.0002

File: urdf/scara.urdf (robot description, URDF)
Before this commit: robot scara, 4 links, 3 joints
Links:
- added link link4; visual mesh filename=package://scara_robot/meshes/link4.STL scale=0.001 0.001 0.001
- link base_link: mass 5 -> None; geometry visual mesh filename=package://scara_robot/meshes/base.STL scale=0.001 0.001 0.001
- link link1: mass 2 -> None; geometry visual mesh filename=package://scara_robot/meshes/link1.STL scale=0.001 0.001 0.001
- link link2: mass 3 -> None; geometry visual mesh filename=package://scara_robot/meshes/link2.STL scale=0.001 0.001 0.001
- link link3: mass 0.3 -> None; geometry visual mesh filename=package://scara_robot/meshes/link3.STL scale=0.001 0.001 0.001
Joints:
- added joint link3_to_link4: type continuous, parent link3, child link4, origin xyz=0 0 -0.047728, axis 0 0 1
- joint base_to_link1: limit lower=-2.094395 upper=2.094395 effort=1000.0 velocity=0.2 -> lower=-2.094395 upper=2.094395 effort=1000.0 velocity=0.02
- joint link1_to_link2: limit lower=-2.268928 upper=2.268928 effort=1000.0 velocity=0.2 -> lower=-2.268928 upper=2.268928 effort=1000.0 velocity=0.02
- joint link2_to_link3: limit lower=-0.15 upper=0.0 effort=1000.0 velocity=0.002 -> lower=-0.15 upper=0.0 effort=1000.0 velocity=0.0002; origin xyz=-0.15 0 0 -> xyz=-0.15 0 0.0
